File: Electronique/PontH_V02.sch (KiCad schematic (older format))
At the start: 6 parts, among them P1 CONN_2, P2 CONN_2, P3 CONN_5

Commit message: carte pont en H V2.1
mais elle a toujours le nom
Parts:
- added C1: CAPAPOL, symbol CAPAPOL
Connections:
- net GND: now also C1.2
- net Vcc: now also C1.1
Changed lines of the file:
@@
-EESchema Schematic File Version 2  date 12/10/2012 19:38:49
+EESchema Schematic File Version 2  date 14/10/2012 16:12:05
 LIBS:power
 LIBS:device
@@
 LIBS:test
 LIBS:vnh2sp30-e
+LIBS:PontH_V02-cache
 EELAYER 25  0
 EELAYER END
@@
 Sheet 1 1
 Title ""
-Date "12 oct 2012"
+Date "14 oct 2012"
 Rev ""
 Comp ""
@@
 Comment4 ""
 $EndDescr
+Wire Wire Line
+	6100 2800 5800 2800
+Connection ~ 7350 2650
+Wire Wire Line
+	7350 2650 6900 2650
+Wire Wire Line
+	6900 2650 6900 2600
 Wire Wire Line
 	8350 2800 8750 2800
@@
 Connection ~ 5950 2800
 Connection ~ 5900 2800
-Wire Wire Line
-	5800 2800 6100 2800
 Connection ~ 6750 4000
 Connection ~ 6750 3900
@@
 	7350 2300 7350 2750
 Wire Wire Line
-	5950 2100 5950 2800
+	5950 2800 5950 2100
 Wire Wire Line
 	5150 3850 4200 3850
@@
 Wire Wire Line
 	8750 3200 8350 3200
+Wire Wire Line
+	6900 2200 6900 2100
+Connection ~ 6900 2100
+$Comp
+L CAPAPOL C1
+U 1 1 507AC439
+P 6900 2400
+F 0 "C1" H 6950 2500 50  0000 L CNN
+F 1 "CAPAPOL" H 6950 2300 50  0000 L CNN
+	1    6900 2400
+	1    0    0    -1
+$EndComp
 Text Label 8350 2900 0    60   ~ 0
 DIAGab
